Commit message: Replace with ROS1 sensor fusion implementation

File: src/robot_description/urdf/automaton.urdf.xacro (robot description, xacro)
@@ -3,5 +3,4 @@
     <xacro:include filename="$(find robot_description)/urdf/automaton.gazebo" />
     <xacro:include filename="$(find robot_description)/urdf/laser.urdf.xacro" />
-    <xacro:include filename="$(find robot_description)/urdf/lidar3d.urdf.xacro" />
     <xacro:property name="PI" value="3.14159"/>
     <xacro:property name="wheel_base" value="0.262"/>
@@ -116,39 +115,15 @@
         <origin xyz="${-wheel_base/2} ${-track_width/2} ${wheel_vertical_offset}" rpy="0.0 0.0 0.0"/>
     </xacro:wheel>
-    <!-- IMU — mounted at chassis centre (internal sensor) -->
-    <link name="imu_link">
-      <inertial>
+    <!-- <link name="imu_link">
+      <interial>
         <mass value="0.001"/>
-        <origin xyz="0 0 0" rpy="0 0 0"/>
-        <inertia ixx="${dummy_inertia}" ixy="0.0" ixz="0.0"
-                 iyy="${dummy_inertia}" iyz="0.0" izz="${dummy_inertia}"/>
-      </inertial>
-    </link>
-    <joint name="imu_joint" type="fixed">
+        <origin xyz="0 0 0" rpy="0 0 0" />
+        <inertia ixx="${dummy_inertia}" ixy="0.0" ixz="0.0" iyy="${dummy_inertia}" iyz="0.0" izz="${dummy_inertia}"/>
+      </interial>
+    </link> -->
+    <!-- <joint name="imu_joint" type="fixed">
       <parent link="chassis_link"/>
       <child link="imu_link"/>
-      <origin xyz="0 0 ${chassis_height/2}" rpy="0 0 0"/>
-    </joint>
-    <!-- GPS — antenna on top-rear of chassis -->
-    <link name="gps_link">
-      <inertial>
-        <mass value="0.001"/>
-        <origin xyz="0 0 0" rpy="0 0 0"/>
-        <inertia ixx="${dummy_inertia}" ixy="0.0" ixz="0.0"
-                 iyy="${dummy_inertia}" iyz="0.0" izz="${dummy_inertia}"/>
-      </inertial>
-      <visual>
-        <origin xyz="0 0 0" rpy="0 0 0"/>
-        <geometry><cylinder radius="0.02" length="0.03"/></geometry>
-        <material name="dark_grey"/>
-      </visual>
-    </link>
-    <joint name="gps_joint" type="fixed">
-      <parent link="chassis_link"/>
-      <child link="gps_link"/>
-      <!-- Top surface of chassis, offset towards rear -->
-      <origin xyz="${-chassis_length/4} 0 ${chassis_height + 0.015}" rpy="0 0 0"/>
-    </joint>
-    <!-- 2D LiDAR front mount -->
+    </joint> -->
     <link name="front_mount"/>
     <joint name="front_mount_joint" type="fixed">
@@ -157,13 +132,11 @@
       <origin xyz="${chassis_length/2.2} 0.0 ${chassis_height}" rpy="0.0 0.0 0.0"/>
     </joint>
-    <!-- 3D LiDAR mount — centre of robot, raised above 2D lidar -->
-    <link name="lidar3d_mount"/>
-    <joint name="lidar3d_mount_joint" type="fixed">
+    <!-- <link name="rear_mount"/>
+    <joint name="rear_mount_joint" type="fixed">
       <parent link="chassis_link"/>
-      <child link="lidar3d_mount"/>
-      <origin xyz="0.0 0.0 ${chassis_height + 0.1}" rpy="0.0 0.0 0.0"/>
-    </joint>
-    <!-- Sensors -->
-    <xacro:hokuyo_ust10 prefix="front" mount="front_mount"/>
-    <xacro:velodyne_vlp16 prefix="top" mount="lidar3d_mount"/>
+      <child link="rear_mount"/>
+      <origin xyz="${-chassis_length/2.2} 0.0 ${chassis_height}" rpy="0.0 0.0 ${-PI}"/>
+    </joint> -->
+    <xacro:hokuyo_ust10 prefix="front" mount="front_mount" />
+    <!-- <xacro:hokuyo_ust10 prefix="rear" mount="rear_mount" /> -->
 </robot>

File: src/robot_description/urdf/laser.urdf.xacro (robot description, xacro)
@@ -1,31 +1,19 @@
 <?xml version="1.0"?>
 <robot xmlns:xacro="http://www.ros.org/wiki/xacro">
-  <!-- ===================================================================
-       Hokuyo UST-10 LiDAR macro — Gazebo Harmonic version.
-       Gazebo Classic used libgazebo_ros_laser.so which embedded ROS
-       publishing directly in the plugin.
-       Gazebo Harmonic separates concerns:
-       1. The <sensor type="gpu_lidar"> block defines the physics/sim sensor.
-          It publishes on a gz topic (e.g. /front_laser/scan).
-       2. ros_gz_bridge (launched in gazebo.launch.py) bridges that gz topic
-          to a ROS2 sensor_msgs/msg/LaserScan topic of the same name.
-       The Sensors system plugin in automaton_world.sdf enables all sensors.
-       =================================================================== -->
-  <xacro:macro name="hokuyo_ust10" params="prefix mount update_rate:=50 sample_size:=720 min_angle:=-2.35619 max_angle:=2.35619 min_range:=0.1 max_range:=30.0 robot_namespace:=/">
+  <xacro:macro name="hokuyo_ust10" params="prefix mount update_rate:=50 sample_size:=720 min_angle:=-2.35619 max_angle:=2.35619 min_range:=0.1 max_range:=30.0 robot_namespace:=/ ">
     <link name="${prefix}_laser">
       <inertial>
-        <mass value="1.1"/>
-        <origin xyz="0 0 0"/>
-        <inertia
-          ixx="${0.0833333 * 1.1 * (0.102*0.102 + 0.152*0.152)}" ixy="0.0" ixz="0.0"
+        <mass value="1.1" />
+        <origin xyz="0 0 0" />
+        <inertia ixx="${0.0833333 * 1.1 * (0.102*0.102 + 0.152*0.152)}" ixy="0.0" ixz="0.0"
           iyy="${0.0833333 * 1.1 * (0.105*0.105 + 0.152*0.152)}" iyz="0.0"
-          izz="${0.0833333 * 1.1 * (0.105*0.105 + 0.102*0.102)}"/>
+          izz="${0.0833333 * 1.1 * (0.105*0.105 + 0.102*0.102)}" />
       </inertial>
       <visual>
         <origin xyz="0.0 0.0 0.0" rpy="0.0 0.0 0.0"/>
         <geometry>
-          <mesh filename="package://robot_description/meshes/hokuyo_ust10_lidar.stl"/>
+          <mesh filename="package://robot_description/meshes/hokuyo_ust10_lidar.stl" />
         </geometry>
-        <material name="dark_grey"/>
+        <material name="dark_grey" />
       </visual>
     </link>
@@ -35,22 +23,11 @@
       <origin xyz="0.0 0.0 0.007" rpy="0.0 0.0 0.0"/>
     </joint>
-    <!-- Gazebo Harmonic: gpu_lidar sensor.
-         Topic is published in the gz domain. The launch file bridges it to ROS2.
-         gz topic:  /${prefix}_laser/scan  (gz.msgs.LaserScan)
-         ROS2 topic: /${prefix}_laser/scan  (sensor_msgs/msg/LaserScan) -->
     <gazebo reference="${prefix}_laser">
-      <visual>
-        <material>
-          <ambient>0.3 0.3 0.3 1</ambient>
-          <diffuse>0.3 0.3 0.3 1</diffuse>
-          <specular>0.1 0.1 0.1 1</specular>
-        </material>
-      </visual>
-      <sensor name="${prefix}_lidar" type="gpu_lidar">
-        <topic>/${prefix}_laser/scan</topic>
-        <gz_frame_id>${prefix}_laser</gz_frame_id>
+      <turnGravityOff>false</turnGravityOff>
+      <sensor type="ray" name="${prefix}_laser">
+        <pose>0 0 0 0 0 0</pose>
+        <visualize>false</visualize>
         <update_rate>${update_rate}</update_rate>
-        <visualize>false</visualize>
-        <lidar>
+        <ray>
           <scan>
             <horizontal>
@@ -71,7 +48,16 @@
             <stddev>0.001</stddev>
           </noise>
-        </lidar>
-        <always_on>1</always_on>
+        </ray>
+        <plugin name="gazebo_ros_laser" filename="libgazebo_ros_laser.so">
+          <topicName>${prefix}_laser/scan</topicName>
+          <frameName>${prefix}_laser</frameName>
+          <robotNamespace>${robot_namespace}</robotNamespace>
+        </plugin>
       </sensor>
+    </gazebo>
+    <gazebo reference="${prefix}_laser">
+      <material>
+        Gazebo/DarkGrey
+      </material>
     </gazebo>
   </xacro:macro>
